File: Hardware/Ogen.sch (KiCad schematic (older format))
At the start: 16 parts, among them J1 Input, U1 TLV70019, U2 PMW3360DM-T2QU, U3 SN74LVC1T45DCK, U4 SN74LVC1T45DCK, U5 SN74LVC1T45DCK, U6 SN74LVC1T45DCK, U7 SN74LVC1T45DCK

Commit message: Fixed major flaw in PMW3360 footprint
Parts:
- U2: footprint Ogen:PMW3360DM-T2QU -> Ogen:IC_PMW3360DM-T2QU
Changed lines of the file:
@@
 F 0 "U2" H 1875 1665 50  0000 C CNN
 F 1 "PMW3360DM-T2QU" H 1875 1574 50  0000 C CNN
-F 2 "Ogen:PMW3360DM-T2QU" H 1900 1550 50  0001 C CNN
+F 2 "Ogen:IC_PMW3360DM-T2QU" H 1900 1550 50  0001 C CNN
 F 3 "" H 1900 1550 50  0001 C CNN
 	1    1850 1150
